Commit message: ros: 젯슨에서 처음 빌드했더니 세 군데서 죽었다 — 전부 "증상이 원인을 안 가리키는" 종류
지금까지 ROS 코드는 **한 번도 빌드된 적이 없었다.** 자체검증 69종이 통과해도
그건 내가 파일을 읽어 계산한 결과일 뿐이라, colcon이 도는지·런치가 뜨는지는
아무것도 말해 주지 않는다. 젯슨(Ubuntu 24.04 noble/arm64)에 올려 실제로 돌렸고,
세 군데서 죽었다. 셋 다 로그가 원인을 안 가리키는 종류였다.

① `entrypoint.sh`의 `set -u`가 ROS를 죽였다
     /opt/ros/jazzy/setup.bash: line 8: AMENT_TRACE_SETUP_FILES: unbound variable
   ROS 환경 스크립트는 미정의 변수 참조를 정상으로 삼는다. 엔트리포인트가 통째로
   죽어 컨테이너가 즉시 종료됐고, colcon은 시작조차 못 했다.

② xacro 매크로 인자를 `len`으로 지었더니 내장 심볼을 덮어썼다
     warning: redefining global symbol: len
   그 자체는 무해한 경고다. 그런데 런치의 `Command` 치환은 **stderr 한 줄을 곧
   실패로** 취급한다 — /robot_description 없음, TF 트리 없음, 링크 0개.
   경고 하나가 로봇 기술 전체를 지운 것이다.
   원인을 고치고(`rod_len`), 증상도 고쳤다(`on_stderr="warn"`) — 앞으로 다른
   경고가 나와도 죽지는 않는다. 진짜 실패면 xacro가 0이 아닌 코드로 끝난다.

③ `Command` 결과를 파라미터로 그냥 줬다
     Unable to parse the value of parameter robot_description as yaml
   URDF는 `<`로 시작해 YAML로도 읽히는 척하다 깨진다. ParameterValue(value_type=str)로
   문자열이라고 명시해야 한다.

그리고 미리 하나 더 — ArUco API가 OpenCV 4.7에서 통째로 바뀌었는데(`ArucoDetector`
도입) 우분투 24.04가 싣는 python3-opencv는 **4.6**이다. 새 API만 쓰면 컨테이너
안에서 AttributeError로 죽고, 증상은 "보정이 안 된다"로만 보인다. 4.6/4.7+ 양쪽에서
도는 `detect_markers()`로 바꿨고, 모듈 최상단에서 cv2.aruco 상수를 읽던 것도 없앴다
(aruco 없는 빌드에서 노드 전체가 죽지 않게).

────────────────────────────────────────────────────────────────
검사를 두 층으로 나눴다 — 아래층이 위층의 구멍을 막는다.

  PC   ros2/tools/ros_selfcheck.py   xacro를 **내가 파싱해** 계산한 값과 대조
                                     구멍: 내가 잘못 읽었으면 검사도 같이 틀린다
  로봇 ros2/tools/bringup_check.sh   진짜 xacro가 펴고, 진짜 robot_state_publisher가
       → tools/tf_check.py           만든 TF를 tf2로 조회해 kinematics.forward()와 대조

두 번째는 팔도 카메라도 필요 없다 — `/joint_states`를 스스로 만들어 쏘기 때문이다.
영점을 잡기 전에도, 팔이 다른 프로세스에 물려 있어도 돌아간다.

실측 결과 (0~2단, 서비스 정지 없이)
  · 6패키지 빌드 1분 12초, 메시지·서비스 5종 생성 확인
  · URDF 링크 13개, TF 트리 base_link → arm_base → tool0
  · RSP가 만든 TF == kinematics.forward()  **7자세 전부 0.000mm**
      전부 0 → (346.0, 0.0, 55.0) · 교시자세(lift=90°) → (0.0, 0.0, 401.0)

곁들여 docker/README.md에 젯슨 실정을 적었다 — Ubuntu 24.04 noble/arm64,
`server`는 docker 그룹이 아니라 sudo가 필요하고, ⚠ **`sudo HOME="$HOME"`을 빠뜨리면**
compose의 `${HOME}` 마운트가 /root가 되어 영점·보정 파일을 엉뚱한 홈에서 찾는다.
RAM 7.4Gi 중 tomato_vision(YOLO)이 2.7Gi를 쓰므로 빌드가 빠듯하다.

Co-Authored-By: Claude Opus 5 (1M context) <noreply@anthropic.com>

File: ros2/src/tomato_description/urdf/so101_arm.xacro (robot description, xacro)
@@ -36,14 +36,19 @@
       </inertial>
     </xacro:macro>
-    <!-- 길이 len짜리 막대를 로컬 +x 방향으로 그린다 -->
-    <xacro:macro name="rod_visual" params="len mname rgba">
+    <!-- 길이 rod_len짜리 막대를 로컬 +x 방향으로 그린다.
+         ⚠ 인자 이름을 `len`으로 두면 안 된다 — xacro의 내장 심볼을 덮어써서
+            `warning: redefining global symbol: len`을 stderr로 뱉는다. 그 자체는
+            무해해 보이지만 런치의 Command 치환이 **stderr 한 줄을 곧 실패로**
+            취급해서 로봇 기술 전체가 안 뜬다(실측: /robot_description 없음,
+            TF 트리 없음, 링크 0개). 증상이 원인을 전혀 안 가리킨다. -->
+    <xacro:macro name="rod_visual" params="rod_len mname rgba">
       <visual>
-        <origin xyz="${len/2} 0 0" rpy="0 ${pi/2} 0"/>
-        <geometry><cylinder radius="${rod_r}" length="${len}"/></geometry>
+        <origin xyz="${rod_len/2} 0 0" rpy="0 ${pi/2} 0"/>
+        <geometry><cylinder radius="${rod_r}" length="${rod_len}"/></geometry>
         <material name="${prefix}m_${mname}"><color rgba="${rgba}"/></material>
       </visual>
       <collision>
-        <origin xyz="${len/2} 0 0" rpy="0 ${pi/2} 0"/>
-        <geometry><cylinder radius="${rod_r}" length="${len}"/></geometry>
+        <origin xyz="${rod_len/2} 0 0" rpy="0 ${pi/2} 0"/>
+        <geometry><cylinder radius="${rod_r}" length="${rod_len}"/></geometry>
       </collision>
     </xacro:macro>
@@ -80,5 +85,5 @@
     <!-- ============ 2. shoulder_lift ============ -->
     <link name="${prefix}upper_arm_link">
-      <xacro:rod_visual len="${l1}" mname="upper" rgba="0.9 0.45 0.2 1"/>
+      <xacro:rod_visual rod_len="${l1}" mname="upper" rgba="0.9 0.45 0.2 1"/>
       <xacro:dummy_inertial m="0.2"/>
     </link>
@@ -92,5 +97,5 @@
     <!-- ============ 3. elbow_flex ============ -->
     <link name="${prefix}forearm_link">
-      <xacro:rod_visual len="${l2}" mname="fore" rgba="0.95 0.7 0.25 1"/>
+      <xacro:rod_visual rod_len="${l2}" mname="fore" rgba="0.95 0.7 0.25 1"/>
       <xacro:dummy_inertial m="0.15"/>
     </link>
@@ -120,5 +125,5 @@
     <!-- ============ 5. wrist_roll ============ -->
     <link name="${prefix}gripper_link">
-      <xacro:rod_visual len="${l3}" mname="grip" rgba="0.55 0.75 0.4 1"/>
+      <xacro:rod_visual rod_len="${l3}" mname="grip" rgba="0.55 0.75 0.4 1"/>
       <xacro:dummy_inertial m="0.1"/>
     </link>
